Commit message: Intro to xacro Variables

File: urdf/my_robot.urdf.xacro (robot description, xacro)
@@ -1,4 +1,12 @@
 <?xml version="1.0"?>
-<robot name="my_robot">
+<robot name="my_robot" xmlns:xacro="https://wiki.ros.org/xacro">
+    <!--    XACRO VARIABLES-->
+    <xacro:property name="base_length" value="0.6" />
+    <xacro:property name="base_width" value="0.4" />
+    <xacro:property name="base_thick" value="0.2" />
+    <xacro:property name="wheel_radius" value="0.1" />
+    <xacro:property name="wheel_length" value="0.05" />
+    <xacro:property name="lidar_radius" value="0.1" />
+    <xacro:property name="lidar_length" value="0.05" />
     <!--    materials-->
     <material name="gray">
@@ -6,5 +14,5 @@
     </material>
     <material name="green">
-        <color rgba="0 0.6 0 1" />
+        <color rgba="0 0.6 0 0.6" />
     </material>
     <material name="white">
@@ -16,7 +24,7 @@
         <visual>
             <geometry>
-                <box size="0.6 0.4 0.2" />
+                <box size="${base_length} ${base_width} ${base_thick}" />
             </geometry>
-            <origin xyz="0 0 0.1" rpy="0 0 0" />
+            <origin xyz="0 0 ${base_thick/2}" rpy="0 0 0" />
             <material name="green" />
         </visual>
@@ -25,5 +33,5 @@
         <visual>
             <geometry>
-                <cylinder radius="0.1" length="0.05" />
+                <cylinder radius="${lidar_radius}" length="${lidar_length}" />
             </geometry>
             <origin xyz="0 0 0" rpy="0 0 0" />
@@ -34,7 +42,7 @@
         <visual>
             <geometry>
-                <cylinder radius="0.1" length="0.05" />
+                <cylinder radius="${wheel_radius}" length="${wheel_length}" />
             </geometry>
-            <origin xyz="0 0 0" rpy="1.57 0 0" />
+            <origin xyz="0 0 0" rpy="${pi/2} 0 0" />
         </visual>
     </link>
@@ -42,7 +50,7 @@
         <visual>
             <geometry>
-                <cylinder radius="0.1" length="0.05" />
+                <cylinder radius="${wheel_radius}" length="${wheel_length}" />
             </geometry>
-            <origin xyz="0 0 0" rpy="1.57 0 0" />
+            <origin xyz="0 0 0" rpy="${pi/2} 0 0" />
         </visual>
     </link>
@@ -50,5 +58,5 @@
         <visual>
             <geometry>
-                <sphere radius="0.05" />
+                <sphere radius="${wheel_radius/2.0}" />
             </geometry>
             <origin xyz="0 0 0" rpy="0 0 0" />
@@ -59,15 +67,15 @@
         <parent link="base_footprint" />
         <child link="base_link" />
-        <origin xyz="0 0 0.1" rpy="0 0 0" />
+        <origin xyz="0 0 ${wheel_radius}" rpy="0 0 0" />
     </joint>
     <joint name="base_lidar_joint" type="fixed">
         <parent link="base_link" />
         <child link="lidar" />
-        <origin xyz="0 0 0.225" rpy="0 0 0" />
+        <origin xyz="0 0 ${base_thick+lidar_length/2}" rpy="0 0 0" />
     </joint>
     <joint name="base_right_wheel_joint" type="continuous">
         <parent link="base_link" />
         <child link="right_wheel" />
-        <origin xyz="-0.15 -0.225  0" rpy="0 0 0" />
+        <origin xyz="-${base_length/4} -${(base_width + wheel_length)/2}  0" rpy="0 0 0" />
         <axis xyz="0 1 0" />
     </joint>
@@ -75,5 +83,5 @@
         <parent link="base_link" />
         <child link="left_wheel" />
-        <origin xyz="-0.15 0.225  0" rpy="0 0 0" />
+        <origin xyz="-${base_length/4} ${(base_width + wheel_length)/2}  0" rpy="0 0 0" />
         <axis xyz="0 1 0" />
     </joint>
@@ -81,5 +89,5 @@
         <parent link="base_link" />
         <child link="caster_wheel" />
-        <origin xyz="0.2 0 -0.05" rpy="0 0 0" />
+        <origin xyz="${base_length/3.0} 0 -${wheel_radius/2.0}" rpy="0 0 0" />
     </joint>
 </robot>

Commit message: Xacro Macros

File: urdf/my_robot.urdf.xacro (robot description, xacro)
@@ -9,4 +9,15 @@
     <xacro:property name="lidar_radius" value="0.1" />
     <xacro:property name="lidar_length" value="0.05" />
+    <!--    XACRO MACROS-->
+    <xacro:macro name="wheel_link" params="prefix" >
+        <link name="${prefix}_wheel_link">
+            <visual>
+                <geometry>
+                    <cylinder radius="${wheel_radius}" length="${wheel_length}" />
+                </geometry>
+                <origin xyz="0 0 0" rpy="${pi/2} 0 0" />
+            </visual>
+        </link>
+    </xacro:macro>
     <!--    materials-->
     <material name="gray">
@@ -39,20 +50,6 @@
         </visual>
     </link>
-    <link name="right_wheel">
-        <visual>
-            <geometry>
-                <cylinder radius="${wheel_radius}" length="${wheel_length}" />
-            </geometry>
-            <origin xyz="0 0 0" rpy="${pi/2} 0 0" />
-        </visual>
-    </link>
-    <link name="left_wheel">
-        <visual>
-            <geometry>
-                <cylinder radius="${wheel_radius}" length="${wheel_length}" />
-            </geometry>
-            <origin xyz="0 0 0" rpy="${pi/2} 0 0" />
-        </visual>
-    </link>
+    <xacro:wheel_link prefix="right" />
+    <xacro:wheel_link prefix="left" />
     <link name="caster_wheel">
         <visual>
@@ -76,5 +73,5 @@
     <joint name="base_right_wheel_joint" type="continuous">
         <parent link="base_link" />
-        <child link="right_wheel" />
+        <child link="right_wheel_link" />
         <origin xyz="-${base_length/4} -${(base_width + wheel_length)/2}  0" rpy="0 0 0" />
         <axis xyz="0 1 0" />
@@ -82,5 +79,5 @@
     <joint name="base_left_wheel_joint" type="continuous">
         <parent link="base_link" />
-        <child link="left_wheel" />
+        <child link="left_wheel_link" />
         <origin xyz="-${base_length/4} ${(base_width + wheel_length)/2}  0" rpy="0 0 0" />
         <axis xyz="0 1 0" />

Commit message: xacro file organization

File: urdf/my_robot.urdf.xacro (robot description, xacro)
@@ -1,90 +1,5 @@
 <?xml version="1.0"?>
 <robot name="my_robot" xmlns:xacro="https://wiki.ros.org/xacro">
-    <!--    XACRO VARIABLES-->
-    <xacro:property name="base_length" value="0.6" />
-    <xacro:property name="base_width" value="0.4" />
-    <xacro:property name="base_thick" value="0.2" />
-    <xacro:property name="wheel_radius" value="0.1" />
-    <xacro:property name="wheel_length" value="0.05" />
-    <xacro:property name="lidar_radius" value="0.1" />
-    <xacro:property name="lidar_length" value="0.05" />
-    <!--    XACRO MACROS-->
-    <xacro:macro name="wheel_link" params="prefix" >
-        <link name="${prefix}_wheel_link">
-            <visual>
-                <geometry>
-                    <cylinder radius="${wheel_radius}" length="${wheel_length}" />
-                </geometry>
-                <origin xyz="0 0 0" rpy="${pi/2} 0 0" />
-            </visual>
-        </link>
-    </xacro:macro>
-    <!--    materials-->
-    <material name="gray">
-        <color rgba="0.7 0.7 0.7 1" />
-    </material>
-    <material name="green">
-        <color rgba="0 0.6 0 0.6" />
-    </material>
-    <material name="white">
-        <color rgba="1 1 1 1" />
-    </material>
-    <!--    links-->
-    <link name="base_footprint" />
-    <link name="base_link">
-        <visual>
-            <geometry>
-                <box size="${base_length} ${base_width} ${base_thick}" />
-            </geometry>
-            <origin xyz="0 0 ${base_thick/2}" rpy="0 0 0" />
-            <material name="green" />
-        </visual>
-    </link>
-    <link name="lidar">
-        <visual>
-            <geometry>
-                <cylinder radius="${lidar_radius}" length="${lidar_length}" />
-            </geometry>
-            <origin xyz="0 0 0" rpy="0 0 0" />
-            <material name="white" />
-        </visual>
-    </link>
-    <xacro:wheel_link prefix="right" />
-    <xacro:wheel_link prefix="left" />
-    <link name="caster_wheel">
-        <visual>
-            <geometry>
-                <sphere radius="${wheel_radius/2.0}" />
-            </geometry>
-            <origin xyz="0 0 0" rpy="0 0 0" />
-        </visual>
-    </link>
-<!--    joints-->
-    <joint name="base_joint" type="fixed">
-        <parent link="base_footprint" />
-        <child link="base_link" />
-        <origin xyz="0 0 ${wheel_radius}" rpy="0 0 0" />
-    </joint>
-    <joint name="base_lidar_joint" type="fixed">
-        <parent link="base_link" />
-        <child link="lidar" />
-        <origin xyz="0 0 ${base_thick+lidar_length/2}" rpy="0 0 0" />
-    </joint>
-    <joint name="base_right_wheel_joint" type="continuous">
-        <parent link="base_link" />
-        <child link="right_wheel_link" />
-        <origin xyz="-${base_length/4} -${(base_width + wheel_length)/2}  0" rpy="0 0 0" />
-        <axis xyz="0 1 0" />
-    </joint>
-    <joint name="base_left_wheel_joint" type="continuous">
-        <parent link="base_link" />
-        <child link="left_wheel_link" />
-        <origin xyz="-${base_length/4} ${(base_width + wheel_length)/2}  0" rpy="0 0 0" />
-        <axis xyz="0 1 0" />
-    </joint>
-    <joint name="base_caster_wheel_joint" type="fixed">
-        <parent link="base_link" />
-        <child link="caster_wheel" />
-        <origin xyz="${base_length/3.0} 0 -${wheel_radius/2.0}" rpy="0 0 0" />
-    </joint>
+    <xacro:include filename="common_properties.xacro" />
+    <xacro:include filename="mobile_base.xacro" />
 </robot>
