Commit message: meshes in xacro file

File: urdf/mobile_base.xacro (robot description, xacro)
@@ -41,5 +41,13 @@
     </link>
     <xacro:wheel_link prefix="right" />
-    <xacro:wheel_link prefix="left" />
+<!--    <xacro:wheel_link prefix="left" />-->
+    <link name="left_wheel_link">
+        <visual>
+            <geometry>
+                <mesh filename="package://my_robot_description/meshes/left_tire.dae" scale="0.001 0.001 0.001"/>
+            </geometry>
+            <origin xyz="0 0 0" rpy="0 0 0" />
+        </visual>
+    </link>
     <link name="caster_wheel">
         <visual>

Commit message: Collision and inertia tags addded.

File: urdf/mobile_base.xacro (robot description, xacro)
@@ -4,5 +4,5 @@
     <xacro:property name="base_length" value="0.6" />
     <xacro:property name="base_width" value="0.4" />
-    <xacro:property name="base_thick" value="0.2" />
+    <xacro:property name="base_height" value="0.2" />
     <xacro:property name="wheel_radius" value="0.1" />
     <xacro:property name="wheel_length" value="0.05" />
@@ -18,4 +18,12 @@
                 <origin xyz="0 0 0" rpy="${pi/2} 0 0" />
             </visual>
+            <collision>
+                <geometry>
+                    <cylinder radius="${wheel_radius}" length="${wheel_length}" />
+                </geometry>
+                <origin xyz="0 0 0" rpy="${pi/2} 0 0" />
+            </collision>
+            <xacro:cylinder_inertia m="1.0" r="${wheel_radius}" l="${wheel_length}"
+                                    xyz="0 0 0" rpy="${pi/2} 0 0" />
         </link>
     </xacro:macro>
@@ -25,9 +33,17 @@
         <visual>
             <geometry>
-                <box size="${base_length} ${base_width} ${base_thick}" />
+                <box size="${base_length} ${base_width} ${base_height}" />
             </geometry>
-            <origin xyz="0 0 ${base_thick/2}" rpy="0 0 0" />
+            <origin xyz="0 0 ${base_height/2}" rpy="0 0 0" />
             <material name="green" />
         </visual>
+        <collision>
+            <geometry>
+                <box size="${base_length} ${base_width} ${base_height}" />
+            </geometry>
+            <origin xyz="0 0 ${base_height/2}" rpy="0 0 0" />
+        </collision>
+        <xacro:box_inertia m="5.0" l="${base_length}" w="${base_width}" h="${base_height}"
+                           xyz="0 0 ${base_height/2}" rpy="0 0 0" />
     </link>
     <link name="lidar">
@@ -49,4 +65,11 @@
             <origin xyz="0 0 0" rpy="0 0 0" />
         </visual>
+        <collision>
+            <geometry>
+                <sphere radius="${wheel_radius/2.0}" />
+            </geometry>
+            <origin xyz="0 0 0" rpy="0 0 0" />
+        </collision>
+        <xacro:sphere_inertia m="1.0" r="${wheel_radius/2.0}" xyz="0 0 0" rpy="0 0 0" />
     </link>
     <!--    joints-->
@@ -59,5 +82,5 @@
         <parent link="base_link" />
         <child link="lidar" />
-        <origin xyz="0 0 ${base_thick+lidar_length/2}" rpy="0 0 0" />
+        <origin xyz="0 0 ${base_height+lidar_length/2}" rpy="0 0 0" />
     </joint>
     <joint name="base_right_wheel_joint" type="continuous">
