Commit message: Collision and inertia tags addded.

File: urdf/common_properties.xacro (robot description, xacro)
@@ -11,3 +11,30 @@
         <color rgba="1 1 1 1" />
     </material>
+    <xacro:macro name="box_inertia" params="m l w h xyz rpy" >
+        <inertial>
+            <origin xyz="${xyz}" rpy="${rpy}" />
+            <mass value="${m}" />
+            <inertia ixx="${m/12*(l*l + h*h)}" ixy="0" ixz="0"
+                     iyy="${m/12*(w*w + l*l)}" iyz="0"
+                     izz="${m/12*(w*w + h*h)}" />
+        </inertial>
+    </xacro:macro>
+    <xacro:macro name="cylinder_inertia" params="m l r xyz rpy" >
+        <inertial>
+            <origin xyz="${xyz}" rpy="${rpy}" />
+            <mass value="${m}" />
+            <inertia ixx="${m/12*(r*r*3 + l*l)}" ixy="0" ixz="0"
+                     iyy="${m/12*(r*r*3 + l*l)}" iyz="0"
+                     izz="${m/2*r*r}" />
+        </inertial>
+    </xacro:macro>
+    <xacro:macro name="sphere_inertia" params="m r xyz rpy" >
+        <inertial>
+            <origin xyz="${xyz}" rpy="${rpy}" />
+            <mass value="${m}" />
+            <inertia ixx="${2/5*m*r*r}" ixy="0" ixz="0"
+                     iyy="${2/5*m*r*r}" iyz="0"
+                     izz="${2/5*m*r*r}" />
+        </inertial>
+    </xacro:macro>
 </robot>

Commit message: Odometry pluging for gazebo simulation

File: urdf/common_properties.xacro (robot description, xacro)
@@ -15,7 +15,7 @@
             <origin xyz="${xyz}" rpy="${rpy}" />
             <mass value="${m}" />
-            <inertia ixx="${m/12*(l*l + h*h)}" ixy="0" ixz="0"
+            <inertia ixx="${m/12*(w*w + h*h)}" ixy="0" ixz="0"
                      iyy="${m/12*(w*w + l*l)}" iyz="0"
-                     izz="${m/12*(w*w + h*h)}" />
+                     izz="${m/12*(w*w + l*l)}" />
         </inertial>
     </xacro:macro>

File: urdf/mobile_base.xacro (robot description, xacro)
@@ -47,13 +47,13 @@
                            xyz="0 0 ${base_height/2}" rpy="0 0 0" />
     </link>
-    <link name="lidar">
-        <visual>
-            <geometry>
-                <cylinder radius="${lidar_radius}" length="${lidar_length}" />
-            </geometry>
-            <origin xyz="0 0 0" rpy="0 0 0" />
-            <material name="white" />
-        </visual>
-    </link>
+<!--    <link name="lidar">-->
+<!--        <visual>-->
+<!--            <geometry>-->
+<!--                <cylinder radius="${lidar_radius}" length="${lidar_length}" />-->
+<!--            </geometry>-->
+<!--            <origin xyz="0 0 0" rpy="0 0 0" />-->
+<!--            <material name="white" />-->
+<!--        </visual>-->
+<!--    </link>-->
     <xacro:wheel_link prefix="right" />
     <xacro:wheel_link prefix="left" />
@@ -79,13 +79,13 @@
         <origin xyz="0 0 ${wheel_radius}" rpy="0 0 0" />
     </joint>
-    <joint name="base_lidar_joint" type="fixed">
-        <parent link="base_link" />
-        <child link="lidar" />
-        <origin xyz="0 0 ${base_height+lidar_length/2}" rpy="0 0 0" />
-    </joint>
+<!--    <joint name="base_lidar_joint" type="fixed">-->
+<!--        <parent link="base_link" />-->
+<!--        <child link="lidar" />-->
+<!--        <origin xyz="0 0 ${base_height+lidar_length/2.0}" rpy="0 0 0" />-->
+<!--    </joint>-->
     <joint name="base_right_wheel_joint" type="continuous">
         <parent link="base_link" />
         <child link="right_wheel_link" />
-        <origin xyz="-${base_length/4} -${(base_width + wheel_length)/2}  0" rpy="0 0 0" />
+        <origin xyz="-${base_length / 4.0} -${(base_width + wheel_length) / 2.0}  0" rpy="0 0 0" />
         <axis xyz="0 1 0" />
     </joint>
@@ -93,5 +93,5 @@
         <parent link="base_link" />
         <child link="left_wheel_link" />
-        <origin xyz="-${base_length/4} ${(base_width + wheel_length)/2}  0" rpy="0 0 0" />
+        <origin xyz="-${base_length / 4.0} ${(base_width + wheel_length)/2.0}  0" rpy="0 0 0" />
         <axis xyz="0 1 0" />
     </joint>
@@ -99,5 +99,5 @@
         <parent link="base_link" />
         <child link="caster_wheel" />
-        <origin xyz="${base_length/3.0} 0 -${wheel_radius/2.0}" rpy="0 0 0" />
+        <origin xyz="${base_length / 3.0} 0 -${wheel_radius / 2.0}" rpy="0 0 0" />
     </joint>
 </robot>

File: urdf/my_robot.urdf.xacro (robot description, xacro)
@@ -1,5 +1,6 @@
 <?xml version="1.0"?>
 <robot name="my_robot" xmlns:xacro="https://wiki.ros.org/xacro">
-    <xacro:include filename="common_properties.xacro" />
-    <xacro:include filename="mobile_base.xacro" />
+    <xacro:include filename="common_properties.xacro" /> <!--INERTIA MACROS -->
+    <xacro:include filename="mobile_base.xacro" /> <!-- URDF DESCRIPTION -->
+    <xacro:include filename="mobile_base_gazebo.xacro" /> <!-- GAZEBO TAGS -->
 </robot>
